File: panels_arena/hallway_panels_arena.sch (KiCad schematic (older format))
At the start: 18 parts, among them J1 DB9, J2 DB9, P1 CONN_5X2, P10 CONN_8, P11 CONN_8, P12 CONN_8, P13 CONN_8, P2 CONN_4X2, P3 CONN_2, P4 CONN_5X2, P5 CONN_4X2, P6 CONN_2, P7 CONN_8, P8 CONN_8, P9 CONN_8, SW1 SWITCH_INV

Commit message: Upgraded hallway arena for kicad 4
Parts:
- removed C1, C2: 10uF, symbol CP1
- removed J1, J2: DB9, symbol DB9
- removed P1, P4: CONN_5X2, symbol CONN_5X2
- removed P10, P11, P12, P13, P7, P8, P9: CONN_8, symbol CONN_8
- removed P2, P5: CONN_4X2, symbol CONN_4X2
- removed P3, P6: CONN_2, symbol CONN_2
- removed SW1: SWITCH_INV, symbol SWITCH_INV
- added C1, C2: 10uF, symbol Device:CP1
- added J1, J2: DB9_Male, symbol Connector:DB9_Male
- added P1, P4: Conn_02x05_Odd_Even, symbol Connector_Generic:Conn_02x05_Odd_Even
- added P10, P11, P12, P13, P7, P8, P9: Conn_01x08, symbol Connector_Generic:Conn_01x08
- added P2, P5: Conn_02x04_Odd_Even, symbol Connector_Generic:Conn_02x04_Odd_Even
- added P3, P6: Barrel_Jack, symbol Connector:Barrel_Jack
- added SW1: SW_SPDT, symbol Switch:SW_SPDT
Connections:
- wire segments 122 -> 139
