File: backlight/hallway_backlight.sch (KiCad schematic (older format))
At the start: 97 parts, among them P1 CONN_2

Commit message: update backligh for kicad 4.
Parts:
- D0,0, D0,1, D0,10, D0,11, D0,12, D0,13, D0,14, D0,15, D0,2, D0,3, D0,4, D0,5, D0,6, D0,7, D0,8, D0,9, D1,0, D1,1, D1,10, D1,11, D1,12, D1,13, D1,14, D1,15, D1,2, D1,3, D1,4, D1,5, D1,6, D1,7, D1,8, D1,9, D2,0, D2,1, D2,10, D2,11, D2,12, D2,13, D2,14, D2,15, D2,2, D2,3, D2,4, D2,5, D2,6, D2,7, D2,8, D2,9, D3,0, D3,1, D3,10, D3,11, D3,12, D3,13, D3,14, D3,15, D3,2, D3,3, D3,4, D3,5, D3,6, D3,7, D3,8, D3,9, D4,0, D4,1, D4,10, D4,11, D4,12, D4,13, D4,14, D4,15, D4,2, D4,3, D4,4, D4,5, D4,6, D4,7, D4,8, D4,9, D5,0, D5,1, D5,10, D5,11, D5,12, D5,13, D5,14, D5,15, D5,2, D5,3, D5,4, D5,5, D5,6, D5,7, D5,8, D5,9: symbol LED -> hallway_backlight-rescue:LED
- P1: symbol CONN_2 -> hallway_backlight-rescue:CONN_2
